File: Keyboard.kicad_pcb (KiCad board)
At the start: 2 copper layers, 404 x 118.3 mm, 220 parts, among them SW2 RotaryEncoder_Switch_MP, U1 MCP23017_SO, U2 MCP23017_SO, U3 Seeeduino Xiao nRF52840

Commit message: Added Mounting Holes to the PCB
Parts:
- added MH1: MountingHole_3.2mm_M3_ISO14580, MountingHole:MountingHole_3.2mm_M3_ISO14580, F.Cu at (402.6, 31.8)
- added MH1: MountingHole_3.2mm_M3_ISO14580, MountingHole:MountingHole_3.2mm_M3_ISO14580, F.Cu at (308.6, 88.9)
- added MH1: MountingHole_3.2mm_M3_ISO14580, MountingHole:MountingHole_3.2mm_M3_ISO14580, F.Cu at (30.5, 141.0)
- added MH1: MountingHole_3.2mm_M3_ISO14580, MountingHole:MountingHole_3.2mm_M3_ISO14580, F.Cu at (138.2, 86.4)
- added MH1: MountingHole_3.2mm_M3_ISO14580, MountingHole:MountingHole_3.2mm_M3_ISO14580, F.Cu at (47.6, 47.6)
- added MH1: MountingHole_3.2mm_M3_ISO14580, MountingHole:MountingHole_3.2mm_M3_ISO14580, F.Cu at (426.7, 141.0)

Commit message: Flipped the Seeed Xiao
Parts:
- C3: moved to F.Cu
- U3: moved to B.Cu
- moved C3 9.33 mm to (414.5, 33.5)
- turned U3 to 180 degrees
Routing:
- net Net-(U1-INTA): track 50.5 -> 71.4 mm
- net +3V3: track 85.7 -> 66.0 mm
- net SCL: track 59.4 -> 78.9 mm
- net Net-(U1-INTB): track 50.0 -> 65.2 mm
- net SDA: track 43.0 -> 57.8 mm
- net GND: track 8.25 -> 3.16 mm, vias 0 -> 1
